File: pcb/jlcpcb/output/combined-panel.kicad_pcb (KiCad board)
At the start: 2 copper layers, 128.5 x 150.1 mm, 150 parts, among them J101 FTSH-106-01-L-D-K, J201 Conn_01x06_MountingPin, J202 FTSH-106-01-L-D-K, SW10 SW_Push, SW11 SW_Push, SW12 SW_Push, SW13 SW_Push, SW15 SW_Push, SW16 SW_Push, SW17 SW_Push, SW18 SW_Push, SW19 SW_Push, SW20 SW_Push, SW22 SW_Push, SW23 SW_Push, SW24 SW_Push, SW25 SW_Push, SW26 SW_Push, SW27 SW_Push, SW28 SW_Push, SW29 SW_Push, SW30 SW_Push, SW31 SW_Push, SW32 SW_Push, SW33 SW_Push, SW34 SW_Push, SW35 SW_Push, SW43 SW_Push, SW44 SW_Push, SW45 SW_Push, SW46 SW_Push, SW47 SW_Push, SW48 SW_Push, SW50 SW_Push, SW51 SW_Push, SW52 SW_Push, SW53 SW_Push, SW54 SW_Push, SW55 SW_Push, SW57 SW_Push, SW58 SW_Push, SW59 SW_Push, SW60 SW_Push, SW61 SW_Push, SW62 SW_Push, SW64 SW_Push, SW65 SW_Push, SW69 SW_Push, SW70 SW_Push, SW8 SW_Push, SW9 SW_Push, U201 XIAO nRF52840 Plus

Commit message: Reduce mouse-bite web for cleaner panel separation
Parts:
- added KiKit_MB_1_8: NPTH, NPTH, F.Cu at (64.9, 86.8)
- added KiKit_MB_2_8: NPTH, NPTH, F.Cu at (97.0, 80.8)
- added KiKit_MB_3_8: NPTH, NPTH, F.Cu at (129.1, 82.8)
- added KiKit_MB_4_8: NPTH, NPTH, F.Cu at (70.9, 91.3)
- added KiKit_MB_5_8: NPTH, NPTH, F.Cu at (103.0, 89.3)
- added KiKit_MB_6_8: NPTH, NPTH, F.Cu at (135.1, 95.3)
- moved KiKit_MB_6_7 0.86 mm to (134.3, 95.3)
- moved KiKit_MB_4_7 0.86 mm to (70.0, 91.3)
- moved KiKit_MB_5_7 0.86 mm to (102.1, 89.3)
- moved KiKit_MB_3_7 0.86 mm to (130.0, 82.8)
- moved KiKit_MB_1_7 0.86 mm to (65.7, 86.8)
- moved KiKit_MB_2_7 0.86 mm to (97.9, 80.8)
- moved KiKit_MB_4_6 0.71 mm to (69.2, 91.3)
- moved KiKit_MB_5_6 0.71 mm to (101.3, 89.3)
- moved KiKit_MB_6_6 0.71 mm to (133.4, 95.3)
- moved KiKit_MB_1_6 0.71 mm to (66.6, 86.8)
- moved KiKit_MB_2_6 0.71 mm to (98.7, 80.8)
- moved KiKit_MB_3_6 0.71 mm to (130.8, 82.8)
- moved KiKit_MB_4_5 0.57 mm to (68.3, 91.3)
- moved KiKit_MB_5_5 0.57 mm to (100.4, 89.3)
- moved KiKit_MB_6_5 0.57 mm to (132.6, 95.3)
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
Commit message: Rename keyboard to FORT-48
Other:
- board text added: "FORT-48"
- board text removed: "kb-1"

Commit message: Rename keyboard to komoro (#54)
Other:
- board text added: "komoro"
- board text removed: "FORT-48"
